Commit message: add gps

File: scout_gazebo/urdf/base.xacro (robot description, xacro)
@@ -41,4 +41,9 @@
     <origin rpy="0 0 0" xyz="-0.03 0 ${base_z_size/2}"/>
     </xacro:imu>
+	<!-- GPS 模块 -->
+	<xacro:include filename="$(find scout_gazebo)/urdf/gps_func.xacro" />
+	<xacro:gps sensor_name="gps" parent_link="base_link">
+	<origin rpy="0 0 0" xyz="-0.03 0 ${base_z_size}"/>
+    </xacro:gps>
     <!-- 机器人导航控制模块 -->
     <xacro:include filename="$(find scout_gazebo)/urdf/move.xacro" />

Commit message: mod

File: scout_gazebo/urdf/base.xacro (robot description, xacro)
@@ -42,8 +42,9 @@
     </xacro:imu>
 	<!-- GPS 模块 -->
+<!--
 	<xacro:include filename="$(find scout_gazebo)/urdf/gps_func.xacro" />
 	<xacro:gps sensor_name="gps" parent_link="base_link">
-	<origin rpy="0 0 0" xyz="-0.03 0 ${base_z_size}"/>
-    </xacro:gps>
+    <origin rpy="0 0 0" xyz="-0.03 0 ${base_z_size*3/2}"/>
+    </xacro:gps>-->
     <!-- 机器人导航控制模块 -->
     <xacro:include filename="$(find scout_gazebo)/urdf/move.xacro" />
@@ -97,3 +98,11 @@
         <origin xyz="${-wheelbase/2} ${-track/2} ${wheel_vertical_offset}" rpy="3.14 0 0" />
     </xacro:scout_wheel_type2>
+    <gazebo>
+	  <plugin name="ground_truth" filename="libgazebo_ros_p3d.so">
+		  <frameName>map</frameName>
+		  <bodyName>base_link</bodyName>
+		  <topicName>gps</topicName>
+		  <updateRate>30.0</updateRate>
+	  </plugin>
+  </gazebo>
 </robot>

File: scout_gazebo/urdf/gps_func.xacro (robot description, xacro)
@@ -1,3 +1,3 @@
-<robot name="sensor" xmlns:xacro="http://www.ros.org/wiki/xacro">
+<robot xmlns:xacro="http://www.ros.org/wiki/xacro">
   <xacro:macro name="gps" params="sensor_name parent_link *origin">
   <xacro:property name="height1" value="0.05" />
@@ -7,9 +7,9 @@
     <xacro:insert_block name="origin" />
     <parent link="${parent_link}"/>
-    <child link="sensor"/>
-    <!--origin xyz="0 0 ${height1 / 2}" /-->
+    <child link="gps_sensor"/>
+    <!--origin xyz="-0.03 0 0.5" rpy="0 0 0" /-->
   </joint>
  <!-- Base Link -->
-  <link name="sensor">
+  <link name="gps_sensor">
     <collision>
       <origin xyz="0 0 ${height1/2}" rpy="0 0 0"/>
@@ -37,13 +37,12 @@
     <color rgba="${255/255} ${108/255} ${10/255} 1.0"/>
   </material>
-        <gazebo reference="sensor">
+        <gazebo reference="gps_sensor">
 	    <material>Gazebo/Orange</material>
-	    <sensor name="gps_sensor" type="gps">
-	    <topic>__default_topic__</topic>
-	    <updateRate>4.0</updateRate>
+	    <sensor name="gps_gazebo" type="gps">
+	    <always_on>true</always_on>
             <plugin name="gazebo_ros_gps" filename="libhector_gazebo_ros_gps.so">
                 <updateRate>4.0</updateRate>
-                <bodyName>sensor</bodyName>
-                <frameId>sensor</frameId>
+                <bodyName>gps_sensor</bodyName>
+                <frameId>gps</frameId>
                 <topicName>gps/fix</topicName>
                 <velocityTopicName>gps/fix_velocity</velocityTopicName>
@@ -57,4 +56,5 @@
                 <velocityDrift>0.001 0.001 0.001</velocityDrift>
                 <velocityGaussianNoise>0.5 0.5 0.5</velocityGaussianNoise>
+                <frameName>gps_sensor</frameName>
             </plugin>
 	</sensor>

File: scout_gazebo/urdf/imu.xacro (robot description, xacro)
@@ -14,5 +14,5 @@
             <child link="imu_base"/>
         </joint>
-        <link name="imu_base">
+        <link name="imu_base"><!--
             <visual>
                 <origin rpy="0 0 0" xyz="0 0 0" />
@@ -30,5 +30,5 @@
                 <origin xyz="0.0 0.0 0" rpy="0.0 0.0 0.0" />
             </collision>
-            <xacro:Box_inertial_matrix m = "${imu_m}" l = "${imu_size}" w = "${imu_size}" h = "${imu_size}"/>
+            <xacro:Box_inertial_matrix m = "${imu_m}" l = "${imu_size}" w = "${imu_size}" h = "${imu_size}"/>-->
         </link>
         <!-- 被引用的link -->
@@ -45,5 +45,5 @@
                 <bodyName>imu_base</bodyName>
                 <updateRateHZ>100.0</updateRateHZ>
-                <gaussianNoise>0.01</gaussianNoise>
+                <gaussianNoise>0.0</gaussianNoise>
                 <xyzOffset>0 0 0</xyzOffset>
                 <rpyOffset>0 0 0</rpyOffset>

File: velodyne_simulator/velodyne_description/urdf/VLP-16.urdf.xacro (robot description, xacro)
@@ -2,5 +2,5 @@
 <robot xmlns:xacro="http://www.ros.org/wiki/xacro" name="VLP-16">
   <xacro:property name="M_PI" value="3.1415926535897931" />
-  <xacro:macro name="VLP-16" params="*origin parent:=base_link name:=velodyne topic:=/velodyne_points organize_cloud:=false hz:=10 lasers:=16 samples:=1875 collision_range:=0.3 min_range:=0.9 max_range:=130.0 noise:=0.0001 min_angle:=-${M_PI} max_angle:=${M_PI} gpu:=false">
+  <xacro:macro name="VLP-16" params="*origin parent:=base_link name:=velodyne topic:=/velodyne_points organize_cloud:=false hz:=10 lasers:=32 samples:=1875 collision_range:=0.3 min_range:=0.9 max_range:=130.0 noise:=0.0001 min_angle:=-${M_PI} max_angle:=${M_PI} gpu:=false">
     <joint name="${name}_base_mount_joint" type="fixed">
       <xacro:insert_block name="origin" />

Commit message: add gps

File: scout_gazebo/urdf/base.xacro (robot description, xacro)
@@ -1,5 +1,5 @@
 <?xml version="1.0"?>
 <robot name="scout_v2"  xmlns:xacro="http://ros.org/wiki/xacro">
-    <xacro:arg name="robot_namespace" default="/" />
+    <xacro:arg name="robot_namespace" default="" />
     <!-- 属性封装 -->
     <xacro:property name="M_PI" value="3.14159"/>
@@ -33,5 +33,5 @@
     <xacro:include filename="$(find scout_gazebo)/urdf/laser_support.xacro" />
     <xacro:include filename="$(find velodyne_description)/urdf/VLP-16.urdf.xacro"/>
-    <xacro:VLP-16 parent="support" name="velodyne" topic="/velodyne_points" organize_cloud="${organize_cloud}" hz="10" samples="440" gpu="${gpu}">
+    <xacro:VLP-16 parent="support" name="velodyne" topic="/velodyne_points" organize_cloud="${organize_cloud}" hz="10" samples="1875" gpu="${gpu}">
           <origin xyz="0 0 ${support_length/2}" rpy="0 0 0" />
     </xacro:VLP-16>
@@ -42,9 +42,5 @@
     </xacro:imu>
 	<!-- GPS 模块 -->
-<!--
 	<xacro:include filename="$(find scout_gazebo)/urdf/gps_func.xacro" />
-	<xacro:gps sensor_name="gps" parent_link="base_link">
-    <origin rpy="0 0 0" xyz="-0.03 0 ${base_z_size*3/2}"/>
-    </xacro:gps>-->
     <!-- 机器人导航控制模块 -->
     <xacro:include filename="$(find scout_gazebo)/urdf/move.xacro" />
@@ -102,5 +98,5 @@
 		  <frameName>map</frameName>
 		  <bodyName>base_link</bodyName>
-		  <topicName>gps</topicName>
+		  <topicName>ground_truth</topicName>
 		  <updateRate>30.0</updateRate>
 	  </plugin>

File: scout_gazebo/urdf/gps_func.xacro (robot description, xacro)
@@ -1,50 +1,11 @@
-<robot xmlns:xacro="http://www.ros.org/wiki/xacro">
-  <xacro:macro name="gps" params="sensor_name parent_link *origin">
-  <xacro:property name="height1" value="0.05" />
-  <xacro:property name="width" value="0.05" />
- <!-- Used for fixing robot to Gazebo 'base_link' -->
-  <joint name="gpstobase" type="fixed">
-    <xacro:insert_block name="origin" />
-    <parent link="${parent_link}"/>
-    <child link="gps_sensor"/>
-    <!--origin xyz="-0.03 0 0.5" rpy="0 0 0" /-->
-  </joint>
- <!-- Base Link -->
-  <link name="gps_sensor">
-    <collision>
-      <origin xyz="0 0 ${height1/2}" rpy="0 0 0"/>
-      <geometry>
-        <box size="${width} ${width} ${height1}"/>
-      </geometry>
-    </collision>
-    <visual>
-      <origin xyz="0 0 ${height1/2}" rpy="0 0 0"/>
-      <geometry>
-        <box size="${width} ${width} ${height1}"/>
-      </geometry>
-      <material name="orange"/>
-    </visual>
-    <inertial>
-      <origin xyz="0 0 1" rpy="0 0 0"/>
-      <mass value="1"/>
-      <inertia
-        ixx="1.0" ixy="0.0" ixz="0.0"
-        iyy="1.0" iyz="0.0"
-        izz="1.0"/>
-    </inertial>
-  </link>
-  <material name="orange">
-    <color rgba="${255/255} ${108/255} ${10/255} 1.0"/>
-  </material>
-        <gazebo reference="gps_sensor">
-	    <material>Gazebo/Orange</material>
-	    <sensor name="gps_gazebo" type="gps">
-	    <always_on>true</always_on>
-            <plugin name="gazebo_ros_gps" filename="libhector_gazebo_ros_gps.so">
+<robot name="sensor" xmlns:xacro="http://www.ros.org/wiki/xacro">
+  <xacro:include filename="$(find scout_gazebo)/urdf/gps_des.xacro"/>
+        <gazebo>
+            <plugin name="gps_sensor" filename="libhector_gazebo_ros_gps.so">
                 <updateRate>4.0</updateRate>
-                <bodyName>gps_sensor</bodyName>
+                <bodyName>sensor</bodyName>
                 <frameId>gps</frameId>
-                <topicName>gps/fix</topicName>
-                <velocityTopicName>gps/fix_velocity</velocityTopicName>
+                <topicName>gps</topicName>
+                <velocityTopicName>gps/velo</velocityTopicName>
                 <referenceLatitude>-30.06022459407145675</referenceLatitude>
                 <referenceLongitude>-51.173913575780311191</referenceLongitude>
@@ -56,8 +17,5 @@
                 <velocityDrift>0.001 0.001 0.001</velocityDrift>
                 <velocityGaussianNoise>0.5 0.5 0.5</velocityGaussianNoise>
-                <frameName>gps_sensor</frameName>
             </plugin>
-	</sensor>
         </gazebo>
-  </xacro:macro>
 </robot>

File: velodyne_simulator/velodyne_description/urdf/VLP-16.urdf.xacro (robot description, xacro)
@@ -2,5 +2,5 @@
 <robot xmlns:xacro="http://www.ros.org/wiki/xacro" name="VLP-16">
   <xacro:property name="M_PI" value="3.1415926535897931" />
-  <xacro:macro name="VLP-16" params="*origin parent:=base_link name:=velodyne topic:=/velodyne_points organize_cloud:=false hz:=10 lasers:=32 samples:=1875 collision_range:=0.3 min_range:=0.9 max_range:=130.0 noise:=0.0001 min_angle:=-${M_PI} max_angle:=${M_PI} gpu:=false">
+  <xacro:macro name="VLP-16" params="*origin parent:=base_link name:=velodyne topic:=/velodyne_points organize_cloud:=false hz:=10 lasers:=16 samples:=1875 collision_range:=0.3 min_range:=0.9 max_range:=130.0 noise:=0.0001 min_angle:=-${M_PI} max_angle:=${M_PI} gpu:=false">
     <joint name="${name}_base_mount_joint" type="fixed">
       <xacro:insert_block name="origin" />
